File: practice_pad/practice_pad.kicad_sch (KiCad schematic)
At the start: 43 parts, among them SW1 SW_Push_45deg, SW10 SW_Push_45deg, SW11 SW_Push_45deg, SW12 SW_Push_45deg, SW13 SW_Push_45deg, SW14 SW_Push_45deg, SW15 SW_Push_45deg, SW16 SW_Push_45deg, SW17 SW_Push_45deg, SW18 SW_Push_45deg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

Commit message: only a few traces left
Connections:
- net at U1.9 (GP8): now also SW10.1, SW14.1, SW17.1, SW2.1, SW6.1
- net at D16.1 (K), D17.1 (K), D18.1 (K): no longer D19.1 (K)
- net at D13.1 (K), D14.1 (K), D15.1 (K): now also D19.1 (K)
Changed lines of the file:
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@@
+	)
+	(junction
+		(at 71.12 40.64)
+		(diameter 0)
+		(color 0 0 0 0)
 	)
 	(junction
@@
 	)
 	(junction
-		(at 93.98 153.67)
-		(diameter 0)
-		(color 0 0 0 0)
-	)
-	(junction
 		(at 88.9 63.5)
 		(diameter 0)
@@
 	)
 	(junction
+		(at 93.98 125.73)
+		(diameter 0)
+		(color 0 0 0 0)
+	)
+	(junction
 		(at 53.34 63.5)
 		(diameter 0)
@@
 	(wire
 		(pts
-			(xy 93.98 153.67) (xy 111.76 153.67)
-		)
-		(stroke
-			(width 0)
-			(type default)
-		)
-	)
-	(wire
-		(pts
 			(xy 58.42 100.33) (xy 76.2 100.33)
 		)
@@
 	(wire
 		(pts
+			(xy 102.87 125.73) (xy 102.87 153.67)
+		)
+		(stroke
+			(width 0)
+			(type default)
+		)
+	)
+	(wire
+		(pts
+			(xy 139.7 66.04) (xy 124.46 66.04)
+		)
+		(stroke
+			(width 0)
+			(type default)
+		)
+	)
+	(wire
+		(pts
 			(xy 58.42 179.07) (xy 93.98 179.07)
 		)
@@
 	(wire
 		(pts
+			(xy 124.46 66.04) (xy 124.46 27.94)
+		)
+		(stroke
+			(width 0)
+			(type default)
+		)
+	)
+	(wire
+		(pts
 			(xy 53.34 40.64) (xy 53.34 63.5)
 		)
@@
 	(wire
 		(pts
+			(xy 71.12 27.94) (xy 124.46 27.94)
+		)
+		(stroke
+			(width 0)
+			(type default)
+		)
+	)
+	(wire
+		(pts
+			(xy 102.87 153.67) (xy 111.76 153.67)
+		)
+		(stroke
+			(width 0)
+			(type default)
+		)
+	)
+	(wire
+		(pts
 			(xy 71.12 87.63) (xy 71.12 113.03)
 		)
@@
 	(wire
 		(pts
+			(xy 71.12 27.94) (xy 71.12 40.64)
+		)
+		(stroke
+			(width 0)
+			(type default)
+		)
+	)
+	(wire
+		(pts
 			(xy 106.68 40.64) (xy 106.68 63.5)
 		)
@@
 		)
 		(stroke
+			(width 0)
+			(type default)
+		)
+	)
+	(wire
+		(pts
+			(xy 93.98 125.73) (xy 102.87 125.73)
+		)
+		(stroke

Commit message: just about done
Connections:
- net at D5.1 (K), D6.1 (K), D7.1 (K)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: now also U1.10 (GP9)
- net at U1.11 (GP10): now also D10.1 (K), D11.1 (K), D12.1 (K), D9.1 (K)
- net at U1.12 (GP11): now also D13.1 (K), D14.1 (K), D15.1 (K), D19.1 (K)
- net at U1.13 (GP12): now also D16.1 (K), D17.1 (K), D18.1 (K)
- net at U1.14 (GP13): now also D20.1 (K), D21.1 (K)
- net at U1.18 (GP27): now also D1.1 (K), D2.1 (K), D3.1 (K), D4.1 (K)
- net at U1.19 (GP28): now also SW11.1, SW15.1, SW18.1, SW21.1, SW3.1, SW7.1
- net at U1.2 (GP1): now also SW1.1, SW13.1, SW16.1, SW20.1, SW5.1, SW9.1
- net at U1.20 (GP29): now also SW12.1, SW19.1, SW4.1, SW8.1

Commit message: Ready to Build
Parts:
- SW1, SW10, SW11, SW12, SW13, SW14, SW15, SW16, SW17, SW18, SW19, SW2, SW20, SW21, SW3, SW4, SW5, SW6, SW7, SW8, SW9: value SW_Push_45deg -> SW_HS
Changed lines of the file:
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@@
 			)
 		)
-		(property "Value" "SW_Push_45deg"
+		(property "Value" "SW_HS"
 			(at 91.44 163.83 0)
 			(effects
@@
 			)
 		)
-		(property "Value" "SW_Push_45deg"
+		(property "Value" "SW_HS"
 			(at 55.88 110.49 0)
 			(effects
@@
 			)
 		)
-		(property "Value" "SW_Push_45deg"
+		(property "Value" "SW_HS"
 			(at 109.22 138.43 0)
 			(effects
@@
 			)
 		)
-		(property "Value" "SW_Push_45deg"
+		(property "Value" "SW_HS"
 			(at 91.44 110.49 0)
 			(effects
@@
 			)
 		)
-		(property "Value" "SW_Push_45deg"
+		(property "Value" "SW_HS"
 			(at 91.44 85.09 0)
 			(effects
@@
 			)
 		)
-		(property "Value" "SW_Push_45deg"
+		(property "Value" "SW_HS"
 			(at 91.44 38.1 0)
 			(effects
@@
 			)
 		)
-		(property "Value" "SW_Push_45deg"
+		(property "Value" "SW_HS"
 			(at 73.66 60.96 0)
 			(effects
@@
 			)
 		)
-		(property "Value" "SW_Push_45deg"
+		(property "Value" "SW_HS"
 			(at 55.88 163.83 0)
 			(effects
@@
 			)
 		)
-		(property "Value" "SW_Push_45deg"
+		(property "Value" "SW_HS"
 			(at 91.44 60.96 0)
 			(effects
@@
 			)
 		)
-		(property "Value" "SW_Push_45deg"
+		(property "Value" "SW_HS"
 			(at 73.66 85.09 0)
 			(effects
@@
 			)
 		)
-		(property "Value" "SW_Push_45deg"
+		(property "Value" "SW_HS"
 			(at 109.22 85.09 0)
 			(effects
@@
 			)
 		)
-		(property "Value" "SW_Push_45deg"
+		(property "Value" "SW_HS"
 			(at 55.88 60.96 0)
 			(effects
@@
 			)
 		)
-		(property "Value" "SW_Push_45deg"
+		(property "Value" "SW_HS"
 			(at 55.88 85.09 0)
 			(effects
@@
 			)
 		)
-		(property "Value" "SW_Push_45deg"
+		(property "Value" "SW_HS"
 			(at 109.22 60.96 0)
 			(effects
@@
 			)
 		)
-		(property "Value" "SW_Push_45deg"
+		(property "Value" "SW_HS"
 			(at 109.22 38.1 0)
 			(effects
@@
 			)
 		)
-		(property "Value" "SW_Push_45deg"
+		(property "Value" "SW_HS"
 			(at 73.66 110.49 0)
 			(effects
@@
 			)
 		)
-		(property "Value" "SW_Push_45deg"
+		(property "Value" "SW_HS"
 			(at 73.66 38.1 0)
 			(effects
@@
 			)
 		)
-		(property "Value" "SW_Push_45deg"
+		(property "Value" "SW_HS"
 			(at 55.88 138.43 0)
 			(effects
@@
 			)
 		)
-		(property "Value" "SW_Push_45deg"
+		(property "Value" "SW_HS"
 			(at 91.44 138.43 0)
 			(effects
@@
 			)
 		)
-		(property "Value" "SW_Push_45deg"
+		(property "Value" "SW_HS"
 			(at 73.66 138.43 0)
 			(effects
@@
 			)
 		)
-		(property "Value" "SW_Push_45deg"
+		(property "Value" "SW_HS"
 			(at 55.88 38.1 0)
 			(effects
