File: scratchpad/scratchpad.kicad_sch (KiCad schematic)
At the start: 0 parts

Commit message: scratchpad complete
Parts:
- added D1, D10, D11, D12, D13, D14, D15, D16, D17, D18, D19, D2, D20, D21, D3, D4, D5, D6, D7, D8, D9: 1N4148W, Diode_SMD:D_SOD-123, symbol Diode:1N4148W
- added J1, J2: Conn_01x09_Socket, Connector_PinSocket_2.54mm:PinSocket_1x09_P2.54mm_Vertical, symbol Connector:Conn_01x09_Socket
- added J3: Conn_01x05_Socket, Connector_PinSocket_2.54mm:PinSocket_1x05_P2.54mm_Vertical, symbol Connector:Conn_01x05_Socket
- added SW1, SW10, SW11, SW13, SW14, SW15, SW16, SW17, SW18, SW2, SW21, SW3, SW4, SW5, SW6, SW7, SW8, SW9: SW_Push_45deg, MX_Hotswap:MX-Hotswap-1U, symbol Switch:SW_Push_45deg
- added SW12, SW19, SW20: SW_Push_45deg, MX_Hotswap:MX-Hotswap-2U-ReversedStabilizers, symbol Switch:SW_Push_45deg
- added U1: RP2040-ZERO_Max, symbol RP2040-ZERO:RP2040-ZERO_Max
Connections:
- new net: D15.2 (A), SW15.2
- new net: D2.2 (A), SW2.2
- new net: D6.2 (A), SW6.2
- new net: D12.2 (A), SW12.2
- new net: D14.2 (A), SW14.2
- new net: D21.2 (A), SW21.2
- new net: D4.2 (A), SW4.2
- new net: D5.2 (A), SW5.2
- new net: D9.2 (A), SW9.2
- new net: D19.2 (A), SW19.2
- new net: D16.2 (A), SW16.2
- new net: D11.2 (A), SW11.2
- new net: D8.2 (A), SW8.2
- new net: D3.2 (A), SW3.2
- new net: D20.2 (A), SW20.2
- new net: D7.2 (A), SW7.2
- new net: D17.2 (A), SW17.2
- new net: D13.2 (A), SW13.2
- new net: D10.2 (A), SW10.2
- new net: D1.2 (A), SW1.2
- new net: D18.2 (A), SW18.2
- new net COL0: J2.7 (Pin_7), SW1.1, SW13.1, SW16.1, SW20.1, SW5.1, SW9.1
- new net COL1: J2.6 (Pin_6), SW10.1, SW14.1, SW17.1, SW2.1, SW6.1
- new net COL2: J1.7 (Pin_7), SW11.1, SW15.1, SW18.1, SW21.1, SW3.1, SW7.1
- new net COL3: J1.6 (Pin_6), SW12.1, SW19.1, SW4.1, SW8.1
- new net ROW0: D1.1 (K), D2.1 (K), D3.1 (K), D4.1 (K), J2.4 (Pin_4)
- new net ROW1: D5.1 (K), D6.1 (K), D7.1 (K), D8.1 (K), J2.5 (Pin_5)
- new net ROW2: D10.1 (K), D11.1 (K), D12.1 (K), D9.1 (K), J1.8 (Pin_8)
- new net ROW3: D13.1 (K), D14.1 (K), D15.1 (K), J2.8 (Pin_8)
- new net ROW4: D16.1 (K), D17.1 (K), D18.1 (K), D19.1 (K), J2.9 (Pin_9)
- new net ROW5: D20.1 (K), D21.1 (K), J1.9 (Pin_9)
